File: TRHCO2_datalogger.sch (EAGLE design)
At the start: 39 parts, among them J6 AMP FCI 10103594-0001LF, U1 ATMEGA328P-MU, U10 TSL2591, U2 FT231XQ-R, U3 DS3234, U7 SHT31/35, U8 MCP1703/3.3V, Y2 SPARKFUN_RESONATORSMD

Commit message: Revert "Initial commit"
This reverts commit c60d50e7691b51f36b2304322911fcaf5220ad07.
Parts:
- removed J6: AMP FCI 10103594-0001LF, SparkFun-Connectors:USB_MICRO-B_HALF_PTH
- removed U$4: 1X7, headers(2mm):1X7
- removed U10: TSL2591, TSL2591:LIGHT_TSL2591
- added B2: JST 2-PH, microbuilder:BATTERY
- added C16, C20: 10uF, microbuilder:CAP_CERAMIC0805-NOOUTLINE
- added C17: 2.2uF, microbuilder:CAP_CERAMIC0805-NOOUTLINE
- added C19: 100uF, rcl:C-USC1210
- added C5: 0.1uF, adafruit:C-USC0402
- added CHRG: ORANGE, microbuilder:LED0805_NOOUTLINE
- added D1: (no value), Adafruit Feather 32u4 Bluefruit LE:MICROBUILDER_DIODE-SCHOTTKYSOD-123
- added DONE1: GREEN, microbuilder:LED0805_NOOUTLINE
- added J3: MicroUSB (5V), SparkFun-Connectors:USB-MICROB
- added JP2: JUMPER-SMT_2_NO_NO-SILK, SparkFun-Jumpers:JUMPER-SMT_2_NO_NO-SILK
- added L2: 6.8uH, microbuilder:INDUCTORTDK_VLC5045
- added LBO: RED, microbuilder:LED0805_NOOUTLINE
- added R33, R41, R42: 1K, microbuilder:RESISTOR0805_NOOUTLINE
- added R34, R36: 200K, microbuilder:RESISTOR0805_NOOUTLINE
- added R35: 1.87M, microbuilder:RESISTOR0805_NOOUTLINE
- added R37: 340K, microbuilder:RESISTOR_0805MP
- added R38: 1.87M, microbuilder:RESISTOR_0805MP
- added R39: 270K, microbuilder:RESISTOR0805_NOOUTLINE
- added R40, R44: 100K, microbuilder:RESISTOR0805_NOOUTLINE
- added R43: 1.0K, microbuilder:RESISTOR0805_NOOUTLINE
- added S2: (no value), SparkFun-Switches:SWITCH-SPDT-SMD-RIGHT-ANGLE
- added T2: MMUN2133LT1G, transistor:MUN2114T1-PNP_DRIVER-SC59-BEC
- added THERM1: 15K, microbuilder:RESISTOR0805_NOOUTLINE
- added U4: TPS61090RSAR, microbuilder:VREG_TPS6103X
- added U5: MCP73871, microbuilder:MCP73871
- added U6: K30-CO2-I2C, K30-CO2-I2C:K30-CO2-I2C
- C4: value 0.1uF -> 1uF; device Adafruit Feather 32u4 Bluefruit LE:MICROBUILDER_CAP_CERAMIC_0402MP -> SparkFun-Capacitors:CAP0805; MPN GRM155R71C104KA88J -> CC0805KKX7R7BB105
Connections:
- removed net D3: U$4.1, U1.PD3
- removed net D4: U$4.2, U1.PD4
- new net 5.0V: C17.1, C19.1, C4.2, R35.2, U4.VOUT, U6.5V
- new net ENABLE: R34.2, U4.EN
- new net LBO: T2.B, U4.LBO
- new net N$14: LBO.A, R33.1
- new net N$28: R35.1, R36.2, U4.FB
- new net N$30: R33.2, T2.C
- new net N$31: R39.1, R40.1, U5.VPCC
- new net N$34: R42.1, U5.STAT2
- new net N$35: R41.1, U5.STAT1/LBO
- new net N$36: R43.2, U5.PROG1
- new net N$37: THERM1.2, U5.THERM
- new net N$38: DONE1.C, R42.2
- new net N$39: CHRG.C, R41.2
- new net N$40: R44.2, U5.PROG3
- new net N$6: L2.2, U4.SW
- new net N$7: R37.2, R38.1, U4.LBI
- new net VBAT: C16.1, C5.1, L2.1, R34.1, R38.2, T2.E, U4.VBAT, U5.VOUT1, U5.VOUT2
- new net VLIPO: C20.1, D1.A, JP2.2, S2.P, U5.VBAT1, U5.VBAT2, U5.VBATSENS
- new net VLIPO_SWITCH: B2.+, JP2.1, S2.S
- net GND: now also B2.-, C16.2, C17.2, C19.2, C20.2, C5.2, J3.GND, LBO.C, R36.1, R37.1, R40.2, R43.1, R44.1, THERM1.1, U4.GND, U4.PGND, U4.SYNC, U5.THERMAL, U5.VSS1, U5.VSS2, U6.GND; no longer J6.GND, U$4.6, U10.GND
- net N$32: now also J3.D-; no longer J6.D-
- net N$33: now also J3.D+; no longer J6.D+
- net SCL: now also U6.SCL; no longer U10.SCL
- net SDA: now also U6.SDA; no longer U10.SDA
- net USB_PWR: now also J3.VBUS; no longer J6.VBUS
- net VBUS: now also CHRG.A, D1.C, DONE1.A, R39.2, U5./TE, U5.CE, U5.PROG2, U5.SEL, U5.VIN1, U5.VIN2
- net VCC: no longer C4.2, U$4.7, U10.VDD
Other:
- note added: "1.0K = 1000mA"
- note added: "10K NTC Thermistor:"
- note added: "2.0K = 500mA"
- note added: "6.8uH power w/2A current"
- note added: "BOOST CONVERTER"
- note added: "Battery Charger"
- note added: "Both grounds must be connected on the PCB at only one point close to the GND pin."
- note added: "CO2"
- note added: "Charge Rate = 1000V/PROG1"
- note added: "No Thermistor:"
- note added: "On/Off Switch"
- note added: "R3 = 1.9Mohm for 5.2V R3 = 1.1Mohm for 3.3V"
- note added: "RT1 = 0, RT2 = 10K"
- note added: "RT1 = TBD, RT2 = TBD"
- note added: "See Pg 15 1st para"
- note added: "v0.3 - May 2017"
- note removed: "0x29"
- note removed: "DS-HCHO"
- note removed: "Light Intensity"
- note removed: "v0.1"
- moved on the sheet: BAT1, C1, C15, C3, C4, C6, D2, JP1, R1, R13, R2, R3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
